File: kicad/classab-amp.kicad_sch (KiCad schematic)
At the start: 81 parts, among them J1 INPUT, Q1 2N5401, Q10 BD140, Q11 BD139, Q12 BD139, Q13 TTC004B, Q14 TTA004B, Q15 IRFP240, Q16 IRFP9240, Q17 IRFP9240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

Commit message: WIP
Parts:
- added C24, C25: 100u, Capacitor_THT:CP_Radial_D4.0mm_P2.00mm, symbol Device:C_Polarized
- added C26: 100p, Capacitor_THT:C_Rect_L7.2mm_W3.0mm_P5.00mm_FKS2_FKP2_MKS2_MKP2, symbol Device:C
- added H1, H2, H3: MountingHole, MountingHole:MountingHole_3.2mm_M3, symbol Mechanical:MountingHole
- added H4: MountingHole, symbol Mechanical:MountingHole
- added R43, R44: 100, Resistor_THT:R_Axial_DIN0207_L6.3mm_D2.5mm_P10.16mm_Horizontal, symbol Device:R
- added R45, R46: 2.2k, Resistor_THT:R_Axial_DIN0204_L3.6mm_D1.6mm_P7.62mm_Horizontal, symbol Device:R
- C6: value 47p -> 100p
- R10, R8: footprint Resistor_THT:R_Axial_DIN0207_L6.3mm_D2.5mm_P2.54mm_Vertical -> Resistor_THT:R_Axial_DIN0204_L3.6mm_D1.6mm_P7.62mm_Horizontal
Connections:
- net B+: now also Q15.1 (G), R25.2, R43.2; no longer C2.1, C5.1, Q1.1 (E), Q9.1 (E), R19.1, R9.1
- net B-: now also R44.2; no longer Q7.1 (E), R11.2, R13.2, R20.2, R7.2
- net PWRGND: now also C24.2, C25.1, R46.2
- net SPEAKER: now also R45.1
- net at Q2.3 (C), Q3.3 (C), Q7.3 (C)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: now also C26.1; no longer C6.1
- new net: C26.2, C6.1, R45.2, R46.1
- new net LP+: C2.1, C24.1, C5.1, Q1.1 (E), Q9.1 (E), R19.1, R43.1, R9.1
- new net LP-: C25.2, Q7.1 (E), R11.2, R13.2, R20.2, R44.1, R7.2
Other:
- moved on the sheet: C6, C9, J3, J4, R22, R23, R25

Commit message: WIP
Connections:
- net B+: no longer Q15.1 (G), R25.2
- new net: Q15.1 (G), R25.2
Other:
- note added: "100V"
Changed lines of the file:
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@@
 	(generator_version "9.0")
 	(paper "A4")
+	(text "100V"
+		(exclude_from_sim no)
+		(at 242.316 87.122 0)
+		(effects
+			(font
+				(size 1.27 1.27)
+			)
+		)
+	)
 	(text "3W"
 		(exclude_from_sim no)
@@
 		)
 	)
+	(text "100V"
+		(exclude_from_sim no)
+		(at 199.39 155.194 0)
+		(effects
+			(font
+				(size 1.27 1.27)
+			)
+		)
+	)
 	(text "BIAS \nTRIM \n"
 		(exclude_from_sim no)
@@
 		)
 	)
+	(text "100V"
+		(exclude_from_sim no)
+		(at 147.32 159.258 0)
+		(effects
+			(font
+				(size 1.27 1.27)
+			)
+		)
+	)
+	(text "100V"
+		(exclude_from_sim no)
+		(at 240.284 154.686 0)
+		(effects
+			(font
+				(size 1.27 1.27)
+			)
+		)
+	)
 	(text "+56V\n"
 		(exclude_from_sim no)
@@
 		)
 	)
+	(text "100V"
+		(exclude_from_sim no)
+		(at 199.136 22.098 0)
+		(effects
+			(font
+				(size 1.27 1.27)
+			)
+		)
+	)
 	(text "3W"
 		(exclude_from_sim no)
@@
 		)
 	)
+	(text "100V"
+		(exclude_from_sim no)
+		(at 158.496 40.132 0)
+		(effects
+			(font
+				(size 1.27 1.27)
+			)
+		)
+	)
 	(text "Non-polarized"
 		(exclude_from_sim no)
@@
 		)
 	)
+	(text "100V"
+		(exclude_from_sim no)
+		(at 240.03 22.606 0)
+		(effects
+			(font
+				(size 1.27 1.27)
+			)
+		)
+	)
 	(text "3W"
 		(exclude_from_sim no)
@@
 	)
 	(junction
-		(at 226.06 44.45)
-		(diameter 0)
-		(color 0 0 0 0)
-	)
-	(junction
 		(at 226.06 146.05)
 		(diameter 0)
@@
 	(wire
 		(pts
-			(xy 226.06 44.45) (xy 226.06 53.34)
+			(xy 226.06 29.21) (xy 226.06 53.34)
 		)
 		(stroke
@@
 		)
 		(stroke
-			(width 0)
-			(type default)
-		)
-	)
-	(wire
-		(pts
-			(xy 226.06 29.21) (xy 226.06 44.45)
-		)
-		(stroke
